File: RubberNugget/v1.0-RubberNugget.sch (KiCad schematic (older format))
At the start: 37 parts, among them J1 USB C 2.0, J2 QWIIC, J3 NeoPixel Breakout, J4 JTAG, J5 Conn_01x04_Male, SW1 Reset, SW2 Reset, SW3 UP, SW4 DOWN, SW5 LEFT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

Commit message: update and re-wire v1.0 alpha
Parts:
- removed J4: JTAG, symbol Connector:Conn_ARM_JTAG_SWD_10
- added J4: Nugget Expansion, Connector_PinHeader_1.27mm:PinHeader_2x08_P1.27mm_Vertical_SMD, symbol Connector_Generic:Conn_02x08_Odd_Even
- added J6: JTAG, Connector_PinHeader_1.27mm:PinHeader_2x05_P1.27mm_Vertical_SMD, symbol Connector_Generic:Conn_02x05_Odd_Even
- C1: footprint (none) -> Capacitor_SMD:C_0603_1608Metric_Pad1.08x0.95mm_HandSolder
- D2: footprint Diode_SMD:D_SOD-123 -> Diode_SMD:D_SOD-323_HandSoldering
- D3: footprint LED_SMD:LED_0603_1608Metric_Pad1.05x0.95mm_HandSolder -> Diode_SMD:D_SOD-323_HandSoldering
- J1: footprint (none) -> Connector_USB:USB_C_Receptacle_Palconn_UTC16-G
- J2: footprint (none) -> Connector_JST:JST_SH_SM04B-SRSS-TB_1x04-1MP_P1.00mm_Horizontal
- J5: value Conn_01x04_Male -> UART; footprint (none) -> Connector_JST:JST_SH_SM04B-SRSS-TB_1x04-1MP_P1.00mm_Horizontal
- R1, R2, R3: footprint (none) -> Resistor_SMD:R_0603_1608Metric_Pad0.98x0.95mm_HandSolder
- U1: footprint Espressif:ESP32-S2-MINI-1 -> Espressif:ESP32-S2-MINI-1_Hand-Soldering
- renumbered C10 to C11
Connections:
- net labels added: A0, A1, A2, A3, A4, A5, A6, MISO, MOSI, SCK
- wire segments 205 -> 238
- no-connect marks 2 -> 12
Other:
- note added: "Microcontroller (ESP32-S2) & Connectors"
- note added: "Nugget D-Pad\n"
- note added: "Nugget Expansion\n"
- note removed: "Connectors\n"
- note removed: "Microcontroller (ESP32-S2)\n"
- note removed: "Nugget D Pad\n"
- moved on the sheet: C10, C11, C5, C6, C7, C8, C9, D3, J1, J2, J3, J5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
